Commit message: new version mppi controller there are somp problems

File: src/bot_description/urdf/bot_v1.camera.xacro (robot description, xacro)
@@ -4,4 +4,5 @@
     name="bot_camera"
     params="
+      mesh_dir:=package://bot_description/meshes
       parent:=chassis_link
       xyz:='0.15 0.0 0.0195'
@@ -30,5 +31,5 @@
         <origin xyz="0 0 0" rpy="0 0 0" />
         <geometry>
-          <mesh filename="package://bot_description/meshes/camera_link.STL" />
+          <mesh filename="${mesh_dir}/camera_link.STL" />
         </geometry>
         <material name="camera_body">

File: src/bot_description/urdf/bot_v1.gazebo.xacro (robot description, xacro)
@@ -28,5 +28,5 @@
   </xacro:if>
   <xacro:if value="$(arg use_camera)">
-    <xacro:bot_camera add_gazebo="true" />
+    <xacro:bot_camera mesh_dir="$(arg mesh_dir)" add_gazebo="true" />
   </xacro:if>
   <gazebo reference="imu_link">

File: src/bot_description/urdf/bot_v1.urdf.xacro (robot description, xacro)
@@ -13,5 +13,5 @@
   </xacro:if>
   <xacro:if value="$(arg use_camera)">
-    <xacro:bot_camera add_gazebo="false" />
+    <xacro:bot_camera mesh_dir="$(arg mesh_dir)" add_gazebo="false" />
   </xacro:if>
 </robot>
