Commit message: Align 3D lidar sim with Unitree L2 datasheet.
Add unitree_4d_lidar_l2.yaml as single source of truth (FOV, range,
128k pts/s, 5.55/216 Hz, 4.5 mm resolution, ±2 cm, 75 mm housing).
Wire parameters into xacro via sim_swerve launch mappings.

File: src/bot_description/urdf/bot_v1.gazebo.xacro (robot description, xacro)
@@ -6,4 +6,16 @@
   <xacro:arg name="use_lidar" default="false" />
   <xacro:arg name="use_camera" default="false" />
+  <!-- Unitree 4D-LiDAR L2 (see config/unitree_4d_lidar_l2.yaml) -->
+  <xacro:arg name="lidar_topic" default="/lidar/points" />
+  <xacro:arg name="lidar_frame_id" default="lidar_link" />
+  <xacro:arg name="lidar_update_rate" default="5.55" />
+  <xacro:arg name="lidar_horizontal_samples" default="591" />
+  <xacro:arg name="lidar_vertical_samples" default="39" />
+  <xacro:arg name="lidar_min_range" default="0.05" />
+  <xacro:arg name="lidar_max_range" default="30.0" />
+  <xacro:arg name="lidar_range_resolution" default="0.0045" />
+  <xacro:arg name="lidar_noise_stddev" default="0.02" />
+  <xacro:arg name="lidar_size_xyz" default="0.075 0.075 0.065" />
+  <xacro:arg name="lidar_mass" default="0.23" />
   <xacro:include filename="bot_v1.core.xacro" />
   <xacro:include filename="bot_v1.lidar.xacro" />
@@ -25,5 +37,17 @@
   <xacro:bot_robot mesh_dir="$(arg mesh_dir)" />
   <xacro:if value="$(arg use_lidar)">
-    <xacro:bot_lidar add_gazebo="true" />
+    <xacro:bot_lidar
+      add_gazebo="true"
+      topic="$(arg lidar_topic)"
+      frame_id="$(arg lidar_frame_id)"
+      update_rate="$(arg lidar_update_rate)"
+      horizontal_samples="$(arg lidar_horizontal_samples)"
+      vertical_samples="$(arg lidar_vertical_samples)"
+      min_range="$(arg lidar_min_range)"
+      max_range="$(arg lidar_max_range)"
+      range_resolution="$(arg lidar_range_resolution)"
+      noise_stddev="$(arg lidar_noise_stddev)"
+      size_xyz="$(arg lidar_size_xyz)"
+      mass="$(arg lidar_mass)" />
   </xacro:if>
   <xacro:if value="$(arg use_camera)">

File: src/bot_description/urdf/bot_v1.lidar.xacro (robot description, xacro)
@@ -1,4 +1,4 @@
 <?xml version="1.0" encoding="utf-8"?>
-<!-- Unitree 4D-LiDAR L2 (sim approximation): 360° x 96° FOV, 0.05-30 m, gpu_lidar -> PointCloud2 -->
+<!-- Unitree 4D-LiDAR L2 — defaults match config/unitree_4d_lidar_l2.yaml (datasheet). -->
 <robot xmlns:xacro="http://www.ros.org/wiki/xacro">
   <xacro:macro
@@ -10,17 +10,22 @@
       add_gazebo:=false
       topic:=/lidar/points
-      update_rate:=10.0
-      horizontal_samples:=360
-      vertical_samples:=32
-      min_angle:=-3.14159
-      max_angle:=3.14159
-      vertical_min_angle:=-0.837758041
-      vertical_max_angle:=0.837758041
+      frame_id:=lidar_link
+      update_rate:=5.55
+      horizontal_samples:=591
+      vertical_samples:=39
+      min_angle:=-3.141592653589793
+      max_angle:=3.141592653589793
+      vertical_min_angle:=-0.8377580409573661
+      vertical_max_angle:=0.8377580409573661
       min_range:=0.05
-      max_range:=30.0">
-    <link name="lidar_link">
+      max_range:=30.0
+      range_resolution:=0.0045
+      noise_stddev:=0.02
+      size_xyz:='0.075 0.075 0.065'
+      mass:=0.23">
+    <link name="${frame_id}">
       <inertial>
         <origin xyz="0 0 0" rpy="0 0 0" />
-        <mass value="0.23" />
+        <mass value="${mass}" />
         <inertia ixx="2e-4" ixy="0.0" ixz="0.0" iyy="2e-4" iyz="0.0" izz="2e-4" />
       </inertial>
@@ -28,8 +33,8 @@
         <origin xyz="0 0 0" rpy="0 0 0" />
         <geometry>
-          <box size="0.075 0.075 0.065" />
+          <box size="${size_xyz}" />
         </geometry>
-        <material name="lidar_gray">
-          <color rgba="0.15 0.15 0.15 1.0" />
+        <material name="unitree_l2_gray">
+          <color rgba="0.12 0.12 0.12 1.0" />
         </material>
       </visual>
@@ -37,5 +42,5 @@
         <origin xyz="0 0 0" rpy="0 0 0" />
         <geometry>
-          <box size="0.075 0.075 0.065" />
+          <box size="${size_xyz}" />
         </geometry>
       </collision>
@@ -44,13 +49,13 @@
       <origin xyz="${xyz}" rpy="${rpy}" />
       <parent link="${parent}" />
-      <child link="lidar_link" />
+      <child link="${frame_id}" />
     </joint>
     <xacro:if value="${add_gazebo}">
-      <gazebo reference="lidar_link">
-        <sensor name="unitree_l2_lidar" type="gpu_lidar">
+      <gazebo reference="${frame_id}">
+        <sensor name="unitree_4d_lidar_l2" type="gpu_lidar">
           <always_on>1</always_on>
           <update_rate>${update_rate}</update_rate>
           <topic>${topic}</topic>
-          <gz_frame_id>lidar_link</gz_frame_id>
+          <gz_frame_id>${frame_id}</gz_frame_id>
           <lidar>
             <scan>
@@ -71,10 +76,10 @@
               <min>${min_range}</min>
               <max>${max_range}</max>
-              <resolution>0.0045</resolution>
+              <resolution>${range_resolution}</resolution>
             </range>
             <noise>
               <type>gaussian</type>
               <mean>0.0</mean>
-              <stddev>0.02</stddev>
+              <stddev>${noise_stddev}</stddev>
             </noise>
           </lidar>

Commit message: both simulation and real__ microros and hardware interface

File: src/bot_description/urdf/bot_v1.gazebo.xacro (robot description, xacro)
@@ -9,18 +9,5 @@
   <xacro:include filename="bot_v1.lidar.xacro" />
   <xacro:include filename="bot_v1.camera.xacro" />
-  <xacro:macro name="ros2_control_position_joint" params="joint_name">
-    <joint name="${joint_name}">
-      <command_interface name="position" />
-      <state_interface name="position" />
-      <state_interface name="velocity" />
-    </joint>
-  </xacro:macro>
-  <xacro:macro name="ros2_control_velocity_joint" params="joint_name">
-    <joint name="${joint_name}">
-      <command_interface name="velocity" />
-      <state_interface name="position" />
-      <state_interface name="velocity" />
-    </joint>
-  </xacro:macro>
+  <xacro:include filename="bot_v1.ros2_control.xacro" />
   <xacro:bot_robot mesh_dir="$(arg mesh_dir)" />
   <xacro:if value="$(arg use_lidar)">
@@ -37,17 +24,7 @@
     </sensor>
   </gazebo>
-  <ros2_control name="bot_gazebo_system" type="system">
-    <hardware>
-      <plugin>gz_ros2_control/GazeboSimSystem</plugin>
-    </hardware>
-    <xacro:ros2_control_position_joint joint_name="f_left_steer" />
-    <xacro:ros2_control_position_joint joint_name="f_right_steer" />
-    <xacro:ros2_control_position_joint joint_name="b_leftsteer" />
-    <xacro:ros2_control_position_joint joint_name="b_rightsteer" />
-    <xacro:ros2_control_velocity_joint joint_name="f_leftwheel" />
-    <xacro:ros2_control_velocity_joint joint_name="f_rightwheel" />
-    <xacro:ros2_control_velocity_joint joint_name="b_leftwheel" />
-    <xacro:ros2_control_velocity_joint joint_name="b_rightwheel" />
-  </ros2_control>
+  <xacro:bot_ros2_control_hardware
+    name="bot_gazebo_system"
+    plugin="gz_ros2_control/GazeboSimSystem" />
   <gazebo>
     <plugin
@@ -65,4 +42,5 @@
       <ros>
         <namespace>/</namespace>
+        <parameter name="use_sim_time">true</parameter>
       </ros>
       <robot_param>robot_description</robot_param>

File: src/bot_description/urdf/bot_v1.urdf.xacro (robot description, xacro)
@@ -1,8 +1,12 @@
 <?xml version="1.0" encoding="utf-8"?>
-<!-- Clean robot description only. Gazebo and ros2_control live in bot_v1.gazebo.xacro. -->
+<!-- Robot model. Optional ros2_control block for real hardware (see enable_ros2_control). -->
 <robot xmlns:xacro="http://www.ros.org/wiki/xacro" name="bot_v1">
   <xacro:arg name="mesh_dir" default="package://bot_description/meshes" />
   <xacro:arg name="use_lidar" default="false" />
   <xacro:arg name="use_camera" default="false" />
+  <xacro:arg name="enable_ros2_control" default="false" />
+  <xacro:arg name="ros2_control_name" default="bot_real_system" />
+  <xacro:arg name="ros2_control_plugin" default="bot_hardware_interface/BotInterface" />
+  <xacro:arg name="use_hw_topics" default="true" />
   <xacro:include filename="bot_v1.core.xacro" />
   <xacro:include filename="bot_v1.lidar.xacro" />
@@ -15,3 +19,10 @@
     <xacro:bot_camera mesh_dir="$(arg mesh_dir)" add_gazebo="false" />
   </xacro:if>
+  <xacro:if value="$(arg enable_ros2_control)">
+    <xacro:include filename="bot_v1.ros2_control.xacro" />
+    <xacro:bot_ros2_control_hardware
+      name="$(arg ros2_control_name)"
+      plugin="$(arg ros2_control_plugin)"
+      use_hw_topics="$(arg use_hw_topics)" />
+  </xacro:if>
 </robot>
